File: DroneBrushlessESC/DroneBrushlessESC.kicad_pcb (KiCad board)
At the start: 2 copper layers, 95 parts, among them J1 UART, J2 Screw_Terminal_01x03, J3 Debug, Q1 CSD17577Q5A, Q2 CSD17577Q5A, Q3 CSD17577Q5A, Q4 CSD17577Q5A, Q5 CSD17577Q5A, Q6 CSD17577Q5A, SW1 PTS815 SJM 250 SMTR LFS, U1 SN74LVC1G11DCKR, U2 M24C02-WMN6TP, U3 STM32G070KBT6, U4 DRV8320SRTVR, U5 INA180A2, U6 INA180A2

Commit message: Finished brushless driver layout
Parts:
- added NT5: NetTie_2, NetTie:NetTie-2_SMD_Pad0.5mm, F.Cu at (150.1, 104.2)
- added NT6: NetTie_2, NetTie:NetTie-2_SMD_Pad0.5mm, F.Cu at (139.1, 115.9)
- added R36: 10K, Resistor_SMD:R_0402_1005Metric, F.Cu at (147.7, 100.7)
- C10, C11, C12, C14, C15, C18, C19, C20, C21, C22, C23, C24, C25, C6, C7, FB1, Q1, Q3, Q5, R10, R13, R14, R16, R17, R25, R27, R28, R29, R3, R30, R7, R8, TP1, TP2, TP3, TP4, TP5, TP6, TP7, TP8, TP9, U5, U6: moved to B.Cu
- TP10: value TR_CSN -> MTR_CSN; moved to B.Cu
- moved J1 241.3 mm to (136.8, 93.0)
- moved R35 240.2 mm to (150.1, 73.9)
- moved D3 236.3 mm to (150.7, 75.2)
- moved TP7 236.1 mm to (144.7, 86.2), turned to 180 degrees
- moved R34 234.6 mm to (157.2, 66.5), turned to 180 degrees
- moved D2 233.8 mm to (154.7, 66.7)
- moved TP4 233.1 mm to (144.8, 91.5), turned to 180 degrees
- moved U2 230.9 mm to (142.2, 85.6)
- moved TP6 230.7 mm to (149.1, 91.3), turned to 180 degrees
- moved TP10 229.9 mm to (150.2, 96.5), turned to 180 degrees
- moved C11 228.8 mm to (142.1, 94.1), turned to 180 degrees
- moved FB1 228.8 mm to (142.0, 92.2)
- moved TP9 226.9 mm to (154.7, 85.8), turned to 180 degrees
- moved R33 224.9 mm to (163.0, 83.5), turned to 180 degrees
- moved TP2 224.5 mm to (153.5, 88.0), turned to 180 degrees
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Connections:
- net Net-(U3-VDD/VDDA) renamed /MCU/VDDA
- Q6 pad 1: GNDPWR -> Net-(U4-SLC)
- Q6 pad 2: GNDPWR -> Net-(U4-SLC)
- Q6 pad 3: GNDPWR -> Net-(U4-SLC)
- TP10 pad 1: TR_CSN -> MTR_CSN
- U3 pad 10: unconnected-(U3-PA3-Pad10) -> EEPROM_WC
- U4 pad 16: GNDPWR -> Net-(U4-SLC)
- U4 pad 31: GNDPWR -> Net-(U4-PGND)
Routing:
- net GND: track 0.00 -> 78.4 mm, vias 0 -> 19
- net FAULT_OUT: track 0.00 -> 62.5 mm, vias 0 -> 5
- net PWM_IN: track 0.00 -> 49.0 mm, vias 0 -> 4
- net +3.3V: track 0.00 -> 46.0 mm, vias 0 -> 14
- net C0_SPI1_MOSI: track 0.00 -> 37.5 mm, vias 0 -> 3
- net GNDPWR: track 0.00 -> 36.2 mm, vias 0 -> 9
- net C0_NRST: track 0.00 -> 35.2 mm, vias 0 -> 6
- net MTR_CURR_A: track 0.00 -> 35.0 mm, vias 0 -> 2
- net C0_SPI1_SCK: track 0.00 -> 32.6 mm, vias 0 -> 2
- net MTR_CURR_B: track 0.00 -> 30.5 mm, vias 0 -> 4
- net UART_RX: track 0.00 -> 30.1 mm, vias 0 -> 2
- net C0_SPI1_MISO: track 0.00 -> 29.4 mm, vias 0 -> 3
- net /Motor/GHC: track 0.00 -> 28.1 mm, vias 0 -> 3
- net MTR_CSN: track 0.00 -> 27.7 mm, vias 0 -> 3
- net /Motor/GHA: track 0.00 -> 27.3 mm, vias 0 -> 3
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- added copper zone on In2.Cu, net +3.3V
- added copper zone on In1.Cu, net GND
- added copper zone on F.Cu, net GNDPWR
- added copper zone on In1.Cu, net GNDPWR
- added copper zone on B.Cu, net MTR_A
- added copper zone on F.Cu, net MTR_A
- added copper zone on B.Cu, net MTR_B
- added copper zone on F.Cu, net MTR_B
- added copper zone on B.Cu, net MTR_C
- added copper zone on F.Cu, net MTR_C
- added copper zone on B.Cu, net VDD
- added copper zone on In2.Cu, net VDD
Other:
- board outline added: 30 x 70 mm
- copper layers 2 -> 4
- board text added: "3.3V"
- board text added: "3.3_PWRGD"
- board text added: "FAULT"
- board text added: "GND"
- board text added: "MISO"
- board text added: "MOSI"
- board text added: "MTR_CSN"
- board text added: "PWM"
- board text added: "RESET"
- board text added: "SCK"
- board text added: "SCL"
- board text added: "SDA"
- board text added: "VDD_PWRGD"
