File: DroneBrushlessESC/DroneBrushlessESC.kicad_sch (KiCad schematic)
At the start: 0 parts

Commit message: Completed schematic for brushless ESC and added needed components to main board.  The plan is to mount the ESCs on the main board using 2.54mm Vert Conn Headers
Other:
- added sheet Debug (Debug.kicad_sch)
- added sheet Power (Power.kicad_sch)
Changed lines of the file:
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@@
 	(paper "A4")
+	(sheet
+		(at 612.14 218.44)
+		(size 250.19 194.31)
+		(exclude_from_sim no)
+		(in_bom yes)
+		(on_board yes)
+		(dnp no)
+		(fields_autoplaced yes)
+		(stroke
+			(width 0.1524)
+			(type solid)
+		)
+		(fill
+			(color 0 0 0 0.0000)
+		)
+		(property "Sheetname" "Debug"
+			(at 612.14 217.7284 0)
+			(effects
+				(font
+					(size 1.27 1.27)
+				)
+				(justify left bottom)
+			)
+		)
+		(property "Sheetfile" "Debug.kicad_sch"
+			(at 612.14 413.3346 0)
+			(effects
+				(font
+					(size 1.27 1.27)
+				)
+				(justify left top)
+			)
+		)
+		(instances
+			(project "DroneBrushlessESC"
+				(path "/3aa1a426-ad7e-4dd6-a1c5-7f97b630afc0"
+					(page "6")
+				)
+			)
+		)
+	)
 	(sheet
 		(at 302.26 0)
@@
 			(project "DroneBrushlessESC"
 				(path "/3aa1a426-ad7e-4dd6-a1c5-7f97b630afc0"
+					(page "4")
+				)
+			)
+		)
+	)
+	(sheet
+		(at 613.41 1.27)
+		(size 248.92 200.66)
+		(exclude_from_sim no)
+		(in_bom yes)
+		(on_board yes)
+		(dnp no)
+		(fields_autoplaced yes)
+		(stroke
+			(width 0.1524)
+			(type solid)
+		)
+		(fill
+			(color 0 0 0 0.0000)
+		)
+		(property "Sheetname" "Power"
+			(at 613.41 0.5584 0)
+			(effects
+				(font
+					(size 1.27 1.27)
+				)
+				(justify left bottom)
+			)
+		)
+		(property "Sheetfile" "Power.kicad_sch"
+			(at 613.41 202.5146 0)
+			(effects
+				(font
+					(size 1.27 1.27)
+				)
+				(justify left top)
+			)
+		)
+		(instances
+			(project "DroneBrushlessESC"
+				(path "/3aa1a426-ad7e-4dd6-a1c5-7f97b630afc0"
 					(page "3")
 				)
@@
 			(project "DroneBrushlessESC"
 				(path "/3aa1a426-ad7e-4dd6-a1c5-7f97b630afc0"
-					(page "4")
-				)
-			)
+					(page "5")
+				)
+			)

Commit message: Finished Schematic for controller
Other:
- title: (none) -> Brushless ESC
Changed lines of the file:
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@@
 	(generator_version "9.0")
 	(paper "A4")
+	(title_block
+		(title "Brushless ESC")
+		(date "2026-02-23")
+		(rev "0-1")
+	)
 	(sheet
 		(at 612.14 218.44)
