File: DroneBrushlessESC/Power.kicad_sch (KiCad schematic)
At the start: 11 parts, among them SW1 PTS815 SJM 250 SMTR LFS, U1 SN74LVC1G11DCKR

Commit message: Finished Schematic for controller
Other:
- title: (none) -> Power
Changed lines of the file:
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@@
 	(generator_version "9.0")
 	(paper "A4")
+	(title_block
+		(title "Power")
+		(date "2026-02-23")
+		(rev "0-1")
+	)
 	(text "AND incomming reset lines for overall MCU reset"
 		(exclude_from_sim no)
