File: Controller/Controller.kicad_pcb (KiCad board)
At the start: 2 copper layers, 68 parts, among them J201 UART, J202 Debug, J203 Battery, Q301 RJK0654DPB-00-J5, SW302 PTS815 SJM 250 SMTR LFS, U301 AP63203WU, U302 SN74LVC1G08DBVR, U401 STM32G070KBT6, U601 THB001P

Commit message: Finished layout for controller, ready to order REV 0-1 PCBs
Parts:
- added C601: 1nf, Capacitor_SMD:C_0402_1005Metric, B.Cu at (152.7, 117.3)
- added C602: 1nf, Capacitor_SMD:C_0402_1005Metric, B.Cu at (153.7, 117.3)
- added C603: 1nf, Capacitor_SMD:C_0402_1005Metric, B.Cu at (146.7, 117.3)
- added R603: 100, Resistor_SMD:R_0402_1005Metric, B.Cu at (154.7, 117.3)
- added R604: 3352T-1-104LF, Library:TRIM_3352T-1-104LF, F.Cu at (114.2, 110.6)
- added R605: 100, Resistor_SMD:R_0402_1005Metric, B.Cu at (145.7, 117.3)
- C401, C402, C403, R401, R402, R403, R404, R405, R406, R407, R408, R409, R410, R411, R412, R413, U401: moved to B.Cu
- R602: value 3352T-1-104LF -> 100; footprint Library:TRIM_3352T-1-104LF -> Resistor_SMD:R_0402_1005Metric; moved to B.Cu
- moved J202 285.3 mm to (118.5, 81.8), turned to 90 degrees
- moved R407 273.7 mm to (140.2, 104.9)
- moved R402 270.8 mm to (140.2, 103.9)
- moved C401 267.7 mm to (147.7, 117.3), turned to -90 degrees
- moved R411 267.2 mm to (149.8, 99.0), turned to -90 degrees
- moved R412 266.2 mm to (150.8, 99.0), turned to -90 degrees
- moved R409 265.5 mm to (148.8, 99.0), turned to -90 degrees
- moved R413 265.3 mm to (151.8, 99.0), turned to 90 degrees
- moved R408 265.3 mm to (148.7, 117.3), turned to -90 degrees
- moved R401 264.3 mm to (146.8, 99.0), turned to 90 degrees
- moved C305 263.6 mm to (119.5, 87.6)
- moved R404 263.6 mm to (147.8, 99.0), turned to -90 degrees
- moved R406 263.4 mm to (150.7, 117.3), turned to -90 degrees
- moved R403 261.4 mm to (149.7, 117.3), turned to 90 degrees
- moved R303 260.8 mm to (119.5, 86.6)
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Connections:
- R602 pad 1: +3.3V -> Net-(R602-Pad1)
- R602 pad 2: POT_VAL -> JSTK_VR2
- U601 pad VR1_2: JSTK_VR1 -> Net-(R603-Pad1)
- U601 pad VR2_2: JSTK_VR2 -> Net-(R602-Pad1)
Routing:
- net UART_RX: track 0.00 -> 62.6 mm, vias 0 -> 1
- net GND: track 0.00 -> 61.2 mm, vias 0 -> 19
- net UART_TX: track 0.00 -> 52.2 mm, vias 0 -> 1
- net C0_NRST: track 0.00 -> 49.8 mm, vias 0 -> 4
- net SWCLK: track 0.00 -> 46.4 mm, vias 0 -> 3
- net Net-(R602-Pad1): track 0.00 -> 43.7 mm, vias 0 -> 1
- net +3.3V: track 0.00 -> 42.8 mm, vias 0 -> 10
- net SWDIO: track 0.00 -> 41.9 mm, vias 0 -> 3
- net Net-(R603-Pad1): track 0.00 -> 39.9 mm, vias 0 -> 1
- net JSTK_BTN: track 0.00 -> 36.2 mm, vias 0 -> 1
- net TR_RXEN: track 0.00 -> 33.5 mm, vias 0 -> 2
- net Net-(R604-Pad2): track 0.00 -> 31.6 mm
- net TR_TXEN: track 0.00 -> 30.3 mm, vias 0 -> 2
- net C0_SPI1_MISO: track 0.00 -> 30.0 mm, vias 0 -> 2
- net TR_IRQ: track 0.00 -> 19.9 mm, vias 0 -> 2
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- added copper zone on In2.Cu, net +3.3V
- added copper zone on F.Cu, net +BATT
- added copper zone on F.Cu, net -BATT
- added copper zone on F.Cu, net /Power/VBAT_SW
- added copper zone on In1.Cu, net GND
- added copper zone on F.Cu, net VBAT_TVS
Other:
- board outline added: 75 x 50 mm
- copper layers 2 -> 4
- board text added: "3.3V"
- board text added: "DEBUG"
- board text added: "DIRECTION"
- board text added: "GND"
- board text added: "NRST"
- board text added: "PWR_GOOD"
- board text added: "RESET"
- board text added: "RX"
- board text added: "SPEED"
- board text added: "SPI_MISO"
- board text added: "SPI_MOSI"
- board text added: "SPI_SCK"
- board text added: "SWCLK"
- board text added: "SWDIO"
- board text added: "TR_CSN"
- board text added: "TX"

Commit message: Swapped polarity of joystick and speed dial so that values line up correctly with desired control.  In short 3.3V on ADC is max speed rather than no speed.
Connections:
- R604 pad 1: +3.3V -> GND
- R604 pad 3: GND -> +3.3V
- U601 pad VR1_1: +3.3V -> GND
- U601 pad VR1_3: GND -> +3.3V
- U601 pad VR2_1: +3.3V -> GND
- U601 pad VR2_3: GND -> +3.3V
Changed lines of the file:
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@@
 			(layers "*.Cu" "*.Mask")
 			(remove_unused_layers no)
-			(net 7 "+3.3V")
+			(net 1 "GND")
 			(pintype "passive")
 			(solder_mask_margin 0.102)
@@
 			(layers "*.Cu" "*.Mask")
 			(remove_unused_layers no)
-			(net 1 "GND")
+			(net 7 "+3.3V")
 			(pintype "passive")
 			(solder_mask_margin 0.102)
@@
 			(layers "*.Cu" "*.Mask")
 			(remove_unused_layers no)
-			(net 7 "+3.3V")
+			(net 1 "GND")
 			(pintype "passive")
 			(solder_mask_margin 0.102)
@@
 			(layers "*.Cu" "*.Mask")
 			(remove_unused_layers no)
-			(net 1 "GND")
+			(net 7 "+3.3V")
 			(pintype "passive")
 			(solder_mask_margin 0.102)
@@
 			(layers "*.Cu" "*.Mask")
 			(remove_unused_layers no)
-			(net 7 "+3.3V")
+			(net 1 "GND")
 			(pintype "passive")
 			(solder_mask_margin 0.102)
@@
 			(layers "*.Cu" "*.Mask")
 			(remove_unused_layers no)
-			(net 1 "GND")
-			(pintype "passive")
-			(solder_mask_margin 0.102)
+			(net 7 "+3.3V")
+			(pintype "passive")
+			(solder_mask_margin 0.102)
